Commit message: Added core XML with basic Robot Colours

File: description/robot.urdf.xacro (robot description, xacro)
@@ -1,5 +1,5 @@
 <?xml version="1.0"?>
 <robot xmlns:xacro="http://www.ros.org/wiki/xacro"  name="robot">
-    <!-- Example link -->
-    <link name="base_link"></link>
+    <!-- URDF : Unified Robot Description Format -->
+    <xacro:include  filename="robot_core.xacro" />
 </robot>
