Commit message: Added Base Robot Geometry

File: description/robot_core.xacro (robot description, xacro)
@@ -14,3 +14,21 @@
         <colour rbga="0 0 0 1" />
     </material>
+    <!-- Easier to set at center of both drive wheels for differential drive robots -->
+    <!-- Rest of the chassis can be referenced to this base link -->
+    <link name="base_link">
+    </link>
+    <joint name="chassis_joint" type="fixed">
+        <parent link="base_link"/>
+        <child link="chassis"/>
+        <origin xyz="0.1 0 0"/>
+    </joint>
+    <link name="chassis">
+        <visual>
+            <origin xyz="0.15 0 0 0.075"/>
+            <geometry>
+                <box size="0.3 0.3 0.15"/>
+            </geometry>
+            <material name="white"/>
+        </visual>
+    </link>
 </robot>

Commit message: Colour was in American and changed 'rbga' to 'rgba'

File: description/robot_core.xacro (robot description, xacro)
@@ -3,14 +3,14 @@
     <!-- URDF : Unified Robot Description Format -->
     <material name="white">
-        <colour rbga="1 1 1 1" />
+        <color rgba="1 1 1 1" />
     </material>
     <material name="orange">
-        <colour rbga="1 0.3 0.1 1" />
+        <color rgba="1 0.3 0.1 1" />
     </material>
     <material name="blue">
-        <colour rbga="0.2 0.2 1 1" />
+        <color rgba="0.2 0.2 1 1" />
     </material>
     <material name="black">
-        <colour rbga="0 0 0 1" />
+        <color rgba="0 0 0 1" />
     </material>
     <!-- Easier to set at center of both drive wheels for differential drive robots -->
@@ -21,9 +21,9 @@
         <parent link="base_link"/>
         <child link="chassis"/>
-        <origin xyz="0.1 0 0"/>
+        <origin xyz="-0.1 0 0"/>
     </joint>
     <link name="chassis">
         <visual>
-            <origin xyz="0.15 0 0 0.075"/>
+            <origin xyz="0.15 0 0.075"/>
             <geometry>
                 <box size="0.3 0.3 0.15"/>

Commit message: Added rough wheel models

File: description/robot_core.xacro (robot description, xacro)
@@ -14,8 +14,10 @@
         <color rgba="0 0 0 1" />
     </material>
+    <!-- BASE LINK -->
     <!-- Easier to set at center of both drive wheels for differential drive robots -->
     <!-- Rest of the chassis can be referenced to this base link -->
     <link name="base_link">
     </link>
+    <!-- CHASSIS -->
     <joint name="chassis_joint" type="fixed">
         <parent link="base_link"/>
@@ -32,3 +34,33 @@
         </visual>
     </link>
+    <!-- LEFT WHEEL LINK -->
+    <joint name="left_wheel_joint" type="continuous">
+        <parent link="base_link"/>
+        <child link="left_wheel"/>
+        <origin xyz="0 0.175 0" rpy="-${pi/2} 0 0"/>
+        <axis xyz="0 0 1"/>
+    </joint>
+    <link name="left_wheel">
+        <visual>
+            <geometry>
+                <cylinder radius="0.05" length="0.04" />
+            </geometry>
+            <material name="blue"/>
+        </visual>
+    </link>
+    <!-- RIGHT WHEEL LINK -->
+    <joint name="right_wheel_joint" type="continuous">
+        <parent link="base_link"/>
+        <child link="right_wheel"/>
+        <origin xyz="0 -0.175 0" rpy="${pi/2} 0 0"/>
+        <axis xyz="0 0 -1"/>
+    </joint>
+    <link name="right_wheel">
+        <visual>
+            <geometry>
+                <cylinder radius="0.05" length="0.04" />
+            </geometry>
+            <material name="blue"/>
+        </visual>
+    </link>
 </robot>

Commit message: Added Caster Wheel and Collision

File: description/robot_core.xacro (robot description, xacro)
@@ -33,4 +33,10 @@
             <material name="white"/>
         </visual>
+        <collision>
+            <origin xyz="0.15 0 0.075"/>
+            <geometry>
+                <box size="0.3 0.3 0.15"/>
+            </geometry>
+        </collision>
     </link>
     <!-- LEFT WHEEL LINK -->
@@ -48,4 +54,9 @@
             <material name="blue"/>
         </visual>
+        <collision>
+            <geometry>
+                <cylinder radius="0.05" length="0.04" />
+            </geometry>
+        </collision>
     </link>
     <!-- RIGHT WHEEL LINK -->
@@ -63,4 +74,28 @@
             <material name="blue"/>
         </visual>
+        <collision>
+            <geometry>
+                <cylinder radius="0.05" length="0.04" />
+            </geometry>
+        </collision>
+    </link>
+        <!-- CASTER WHEEL LINK -->
+    <joint name="caster_wheel_joint" type="continuous">
+        <parent link="chassis"/>
+        <child link="caster_wheel"/>
+        <origin xyz="0.24 0 0"/>
+    </joint>
+    <link name="caster_wheel">
+        <visual>
+            <geometry>
+                <sphere radius="0.05"/>
+            </geometry>
+            <material name="black"/>
+        </visual>
+        <collision>
+            <geometry>
+                <sphere radius="0.05"/>
+            </geometry>
+        </collision>
     </link>
 </robot>

Commit message: Added inertia details to links

File: description/robot_core.xacro (robot description, xacro)
@@ -1,4 +1,5 @@
 <?xml version="1.0"?>
 <robot xmlns:xacro="http://www.ros.org/wiki/xacro" >
+    <xacro:include  filename="inertial_marcos.xacro" />
     <!-- URDF : Unified Robot Description Format -->
     <material name="white">
@@ -39,4 +40,7 @@
             </geometry>
         </collision>
+        <xacro:inertial_box mass="0.5" x="0.3" y="0.3" z="0.15">
+            <origin xyz="0.15 0 0.075" rpy="0 0 0"/>
+        </xacro:inertial_box>
     </link>
     <!-- LEFT WHEEL LINK -->
@@ -59,4 +63,7 @@
             </geometry>
         </collision>
+        <xacro:inertial_cylinder mass="0.1" length="0.04" radius="0.05">
+            <origin xyz="0 0 0" rpy="0 0 0"/>
+        </xacro:inertial_cylinder>
     </link>
     <!-- RIGHT WHEEL LINK -->
@@ -79,4 +86,7 @@
             </geometry>
         </collision>
+        <xacro:inertial_cylinder mass="0.1" length="0.04" radius="0.05">
+            <origin xyz="0 0 0" rpy="0 0 0"/>
+        </xacro:inertial_cylinder>
     </link>
         <!-- CASTER WHEEL LINK -->
@@ -98,4 +108,7 @@
             </geometry>
         </collision>
+        <xacro:inertial_sphere mass="0.1" radius="0.05">
+            <origin xyz="0 0 0" rpy="0 0 0"/>
+        </xacro:inertial_sphere>
     </link>
 </robot>

Commit message: Added rviz config

File: description/robot_core.xacro (robot description, xacro)
@@ -91,5 +91,5 @@
     </link>
         <!-- CASTER WHEEL LINK -->
-    <joint name="caster_wheel_joint" type="continuous">
+    <joint name="caster_wheel_joint" type="fixed">
         <parent link="chassis"/>
         <child link="caster_wheel"/>
